Commit message: Adding Inertia tags and installing gazebo

File: description/robot_core.xacro (robot description, xacro)
@@ -1,4 +1,5 @@
 <?xml version="1.0"?>
 <robot xmlns:xacro="http://www.ros.org/wiki/xacro" >
+    <xacro:include filename="Inertial_macros.xacro"/>
     <xacro:property name="chassis_length" value="0.3"/>
     <xacro:property name="chassis_width" value="0.2"/>
@@ -49,4 +50,7 @@
             </geometry>
         </collision>
+        <xacro:inertial_box mass="0.5" x="${chassis_length}" y="${chassis_width}" z="${chassis_height}">
+            <origin xyz="${chassis_length/2} 0 ${chassis_height/2}" rpy="0 0 0"/>
+        </xacro:inertial_box>
     </link>
     <gazebo reference="chassis">
@@ -72,4 +76,7 @@
             </geometry>
         </collision>
+                <xacro:inertial_cylinder mass="${wheel_mass}" length="${wheel_thickness}" radius="${wheel_radius}">
+            <origin xyz="0 0 0" rpy="0 0 0"/>
+        </xacro:inertial_cylinder>
     </link>
     <gazebo reference="left_Fwheel">
@@ -94,4 +101,7 @@
             </geometry>
         </collision>
+                <xacro:inertial_cylinder mass="${wheel_mass}" length="${wheel_thickness}" radius="${wheel_radius}">
+            <origin xyz="0 0 0" rpy="0 0 0"/>
+        </xacro:inertial_cylinder>
     </link>
     <gazebo reference="left_Bwheel">
@@ -117,4 +127,7 @@
             </geometry>
         </collision>
+                <xacro:inertial_cylinder mass="${wheel_mass}" length="${wheel_thickness}" radius="${wheel_radius}">
+            <origin xyz="0 0 0" rpy="0 0 0"/>
+        </xacro:inertial_cylinder>
     </link>
     <gazebo reference="right_Fwheel">
@@ -139,4 +152,7 @@
             </geometry>
         </collision>
+                <xacro:inertial_cylinder mass="${wheel_mass}" length="${wheel_thickness}" radius="${wheel_radius}">
+            <origin xyz="0 0 0" rpy="0 0 0"/>
+        </xacro:inertial_cylinder>
     </link>
     <gazebo reference="right_Bwheel">

Commit message: mapping online

File: description/robot_core.xacro (robot description, xacro)
@@ -57,4 +57,12 @@
         <material>Gazebo/Orange</material>
     </gazebo>
+    <!-- BASE FOOTPRINT -->
+    <joint name="base_footprint_joint" type="fixed">
+        <parent link="base_link"/>
+        <child link="base_footprint"/>
+        <origin xyz="0 0 0" rpy="0 0 0" />
+    </joint>
+    <link name="base_footprint">
+    </link>
    <!-- LEFT WHEEL LINK -->
     <joint name="left_F_wheel_joint" type="continuous">
