Commit message: adding gazebo model and controller for robot arm

File: description/arm_model.xacro (robot description, xacro)
@@ -16,13 +16,22 @@
   <xacro:property name="gripper_h" value="0.1" />
   <xacro:property name="gripper_m" value="0.1" />
+  <xacro:macro name="default_transmission" params="joint_name">
+    <transmission name="transmission_${joint_name}">
+      <plugin>transmission_interface/SimpleTransmission</plugin>
+      <actuator name="motor_${joint_name}" role="actuator1" />
+      <joint name="${joint_name}" role="joint1">
+        <mechanical_reduction>1.0</mechanical_reduction>
+      </joint>
+    </transmission>
+  </xacro:macro>
   <link name="static_base_link">
     <visual>
       <geometry>
-        <box size="${base_l} ${base_w} ${base_h}" />
+        <box size="${base_l+0.2} ${base_w+0.2} ${base_h}" />
       </geometry>
       <origin xyz="0 0 ${base_h/2.0}" rpy="0 0 0" />
       <material name="grey" />
     </visual>
-    <xacro:inertia_box m="${base_m}" l="${base_l}" w="${base_w}" h="${base_h}"
+    <xacro:inertia_box m="${3*base_m}" l="${base_l}" w="${base_w}" h="${base_h}"
       xyz="0 0 ${-base_h/2.0}" rpy="0 0 0" />
     <collision>
@@ -53,5 +62,5 @@
     <axis xyz="0 0 1" />
     <origin xyz="0 0 ${base_h}" rpy="0 0 0" />
-    <limit effort="1000.0" upper="${pi}" lower="${-pi}" velocity="0.5" />
+    <limit effort="1000.0" upper="${PI/2.0}" lower="${-PI/2.0}" velocity="0.5" />
     <parent link="static_base_link" />
     <child link="arm_base_link" />
@@ -80,15 +89,39 @@
     <axis xyz="0 1 0" />
     <origin xyz="0 ${arm_w/2} ${base_h}" rpy="0 0 0" />
-    <limit effort="1000.0" upper="${pi}" lower="${-pi}" velocity="0.5" />
+    <limit effort="1000.0" upper="${PI/2.0}" lower="${-PI/2.0}" velocity="0.5" />
     <parent link="arm_base_link" />
     <child link="arm_1_link" />
   </joint>
-  <xacro:arm_links prefix="arm_2" color="yellow" y_offset="${-arm_w/2.0}"/>
+  <xacro:arm_links prefix="arm_2" color="yellow" y_offset="${-arm_w/2.0}" />
   <joint name="arm1_arm2_joint" type="revolute">
     <axis xyz="0 1 0" />
     <origin xyz="0 ${-arm_w/2} ${arm_h-0.1}" rpy="0 0 0" />
-    <limit effort="1000.0" upper="${pi}" lower="${-pi}" velocity="0.5" />
+    <limit effort="1000.0" upper="${PI/2.0}" lower="${-PI/2.0}" velocity="0.5" />
     <parent link="arm_1_link" />
     <child link="arm_2_link" />
+  </joint>
+  <link name="arm_3_link">
+    <visual>
+      <geometry>
+        <box size="${arm_l} ${arm_w} ${arm_h/3}" />
+      </geometry>
+      <origin xyz="0 0 ${arm_h/6}" rpy="0 0 0"></origin>
+      <material name="orange" />
+    </visual>
+    <collision>
+      <origin xyz="0 0 ${arm_h/6}" rpy="0 0 0"></origin>
+      <geometry>
+        <box size="${arm_l} ${arm_w} ${arm_h/3}" />
+      </geometry>
+    </collision>
+    <xacro:inertia_box m="${arm_m}" l="${arm_l}" w="${arm_w}" h="${arm_h/3}"
+      xyz="0 0 ${-arm_h/6.0}" rpy="0 0 0" />
+  </link>
+  <joint name="arm2_arm3_joint" type="revolute">
+    <axis xyz="0 1 0" />
+    <origin xyz="0 ${arm_w/2} ${arm_h-0.05}" rpy="0 0 0" />
+    <limit effort="1000.0" upper="${PI/2.0}" lower="${-PI/2.0}" velocity="0.5" />
+    <parent link="arm_2_link" />
+    <child link="arm_3_link" />
   </joint>
   <link name="wrist_link">
@@ -97,9 +130,9 @@
         <cylinder radius="${wrist_r}" length="${wrist_l}" />
       </geometry>
-      <origin xyz="0 0 0" rpy="0 0 0"/>
+      <origin xyz="0 0 0" rpy="0 0 0" />
       <material name="blue" />
     </visual>
     <collision>
-      <origin xyz="0 0 0" rpy="0 0 0"/>
+      <origin xyz="0 0 0" rpy="0 0 0" />
       <geometry>
         <cylinder radius="${wrist_r}" length="${wrist_l}" />
@@ -109,10 +142,52 @@
       xyz="0 0 ${-arm_h/2.0}" rpy="0 0 0" />
   </link>
-  <joint name="arm1_wrist_joint" type="revolute">
+  <joint name="arm3_wrist_joint" type="revolute">
     <axis xyz="0 0 1" />
-    <origin xyz="0 ${-arm_w/2.0} ${arm_h}" rpy="0 0 0" />
-    <limit effort="1000.0" upper="${pi}" lower="${-pi}" velocity="0.5" />
-    <parent link="arm_2_link" />
+    <origin xyz="0 0 ${arm_h/3}" rpy="0 0 0" />
+    <limit effort="1000.0" upper="${PI/2.0}" lower="${-PI/2.0}" velocity="0.5" />
+    <parent link="arm_3_link" />
     <child link="wrist_link" />
   </joint>
+  <xacro:macro name="gripper_links" params="prefix y_offset">
+    <link name="${prefix}_link">
+      <visual>
+        <geometry>
+          <box size="${gripper_l} ${gripper_w} ${gripper_h}" />
+        </geometry>
+        <origin xyz="0 ${y_offset} ${gripper_h/2}" rpy="0 0 0"></origin>
+        <material name="grey" />
+      </visual>
+      <collision>
+        <origin xyz="0 0 ${gripper_h/2}" rpy="0 0 0"></origin>
+        <geometry>
+          <box size="${gripper_l} ${gripper_w} ${gripper_h}" />
+        </geometry>
+      </collision>
+      <xacro:inertia_box m="${gripper_m}" l="${gripper_l}" w="${gripper_w}" h="${gripper_h}"
+        xyz="0 0 ${-gripper_h/2.0}" rpy="0 0 0" />
+    </link>
+  </xacro:macro>
+  <xacro:gripper_links prefix="gripper_l" y_offset="${-gripper_w/2}" />
+  <xacro:gripper_links prefix="gripper_r" y_offset="${gripper_w/2}" />
+  <joint name="wrist_gripr_joint" type="prismatic">
+    <axis xyz="0 1 0" />
+    <origin xyz="0 0 ${wrist_l}" rpy="0 0 0" />
+    <limit effort="1000.0" upper="0" lower="-0.3" velocity="0.5" />
+    <parent link="wrist_link" />
+    <child link="gripper_r_link" />
+    <mimic joint="wrist_gripl_joint" multiplier="-1"/>
+  </joint>
+  <joint name="wrist_gripl_joint" type="prismatic">
+    <axis xyz="0 1 0" />
+    <origin xyz="0 0 ${wrist_l}" rpy="0 0 0" />
+    <limit effort="1000.0" upper="0.3" lower="0" velocity="0.5" />
+    <parent link="wrist_link" />
+    <child link="gripper_l_link" />
+  </joint>
+  <xacro:default_transmission joint_name="bases_joint" />
+  <xacro:default_transmission joint_name="base_arm1_joint" />
+  <xacro:default_transmission joint_name="arm1_arm2_joint" />
+  <xacro:default_transmission joint_name="arm2_arm3_joint" />
+  <xacro:default_transmission joint_name="arm3_wrist_joint" />
+  <xacro:default_transmission joint_name="wrist_gripl_joint" />
 </robot>

File: description/common_properties.xacro (robot description, xacro)
@@ -16,4 +16,5 @@
         <color rgba="0.7 0.4 0.0 1" />
     </material>
+    <xacro:property name="PI" value="3.14159"/>
     <xacro:macro name="inertia_box" params="m l w h xyz rpy">
         <inertial>

File: description/robot_arm.urdf.xacro (robot description, xacro)
@@ -3,3 +3,5 @@
     <xacro:include filename="common_properties.xacro" />
     <xacro:include filename="arm_model.xacro" />
+    <xacro:include filename="arm_gazebo.xacro" />
+    <xacro:include filename="ros2_control.xacro" />
 </robot>
