Commit message: changing robot config and adding gripping reference

File: simple_arm/robo_arm/description/arm_model.xacro (robot description, xacro)
@@ -5,14 +5,14 @@
   <xacro:property name="base_h" value="0.05" />
   <xacro:property name="base_m" value="0.3" />
-  <xacro:property name="arm_l" value="0.05" />
-  <xacro:property name="arm_w" value="0.05" />
-  <xacro:property name="arm_h" value="0.3" />
+  <xacro:property name="arm_l" value="0.03" />
+  <xacro:property name="arm_w" value="0.03" />
+  <xacro:property name="arm_h" value="0.15" />
   <xacro:property name="arm_m" value="0.3" />
   <xacro:property name="wrist_r" value="0.025" />
   <xacro:property name="wrist_l" value="0.01" />
   <xacro:property name="wrist_m" value="0.1" />
-  <xacro:property name="gripper_l" value="0.05" />
-  <xacro:property name="gripper_w" value="0.05" />
-  <xacro:property name="gripper_h" value="0.1" />
+  <xacro:property name="gripper_l" value="0.04" />
+  <xacro:property name="gripper_w" value="0.04" />
+  <xacro:property name="gripper_h" value="0.08" />
   <xacro:property name="gripper_m" value="0.1" />
   <xacro:macro name="default_transmission" params="joint_name">
@@ -33,5 +33,5 @@
       <material name="grey" />
     </visual>
-    <xacro:inertia_box m="${3*base_m}" l="${base_l}" w="${base_w}" h="${base_h}"
+    <xacro:inertia_box m="${10*base_m}" l="${base_l}" w="${base_w}" h="${base_h}"
       xyz="0 0 ${-base_h/2.0}" rpy="0 0 0" />
     <collision>
@@ -96,6 +96,6 @@
   <joint name="arm1_arm2_joint" type="revolute">
     <axis xyz="0 1 0" />
-    <origin xyz="0 ${-arm_w/2} ${arm_h-0.1}" rpy="0 0 0" />
-    <limit effort="1000.0" upper="${PI/2.0}" lower="${-PI/2.0}" velocity="0.5" />
+    <origin xyz="0 ${-arm_w/2} ${arm_h-0.03}" rpy="0 0 0" />
+    <limit effort="1000.0" upper="${PI}" lower="${-PI/2.0}" velocity="0.5" />
     <parent link="arm_1_link" />
     <child link="arm_2_link" />
@@ -120,5 +120,5 @@
   <joint name="arm2_arm3_joint" type="revolute">
     <axis xyz="0 1 0" />
-    <origin xyz="0 ${arm_w/2} ${arm_h-0.05}" rpy="0 0 0" />
+    <origin xyz="0 ${arm_w/2} ${arm_h-0.03}" rpy="0 0 0" />
     <limit effort="1000.0" upper="${PI/2.0}" lower="${-PI/2.0}" velocity="0.5" />
     <parent link="arm_2_link" />
@@ -159,5 +159,5 @@
       </visual>
       <collision>
-        <origin xyz="0 0 ${gripper_h/2}" rpy="0 0 0"></origin>
+        <origin xyz="0 ${y_offset} ${gripper_h/2}" rpy="0 0 0"></origin>
         <geometry>
           <box size="${gripper_l} ${gripper_w} ${gripper_h}" />
@@ -168,6 +168,6 @@
     </link>
   </xacro:macro>
-  <xacro:gripper_links prefix="gripper_l" y_offset="${-gripper_w/2}" />
-  <xacro:gripper_links prefix="gripper_r" y_offset="${gripper_w/2}" />
+  <xacro:gripper_links prefix="gripper_l" y_offset="${gripper_w/2}" />
+  <xacro:gripper_links prefix="gripper_r" y_offset="${-gripper_w/2}" />
   <joint name="wrist_gripr_joint" type="prismatic">
     <axis xyz="0 1 0" />
